File: kicad_project/digitizer/MCU.kicad_sch (KiCad schematic)
At the start: 20 parts, among them J401 Conn_02x05_Odd_Even

Commit message: updated annotations
Parts:
- gave numbers to parts that had none: 17
Changed lines of the file:
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@@
   (symbol (lib_id "power:GND") (at 234.95 39.37 0) (unit 1)
     (in_bom yes) (on_board yes)
-    (property "Reference" "#PWR?" (id 0) (at 234.95 45.72 0)
+    (property "Reference" "#PWR0403" (id 0) (at 234.95 45.72 0)
       (effects (font (size 1.27 1.27)) hide)
     )
@@
   (symbol (lib_id "2022-01-19_19-47-49:ATSAM4E8EA-AN") (at 167.64 27.94 0) (unit 2)
     (in_bom yes) (on_board yes) (fields_autoplaced)
-    (property "Reference" "U?" (id 0) (at 187.96 16.51 0)
+    (property "Reference" "U401" (id 0) (at 187.96 16.51 0)
       (effects (font (size 1.524 1.524)))
     )
@@
   (symbol (lib_id "Device:C_Small") (at 234.95 52.07 0) (unit 1)
     (in_bom yes) (on_board yes)
-    (property "Reference" "C?" (id 0) (at 236.22 49.53 0)
+    (property "Reference" "C409" (id 0) (at 236.22 49.53 0)
       (effects (font (size 1.27 1.27)) (justify left))
     )
@@
   (symbol (lib_id "Device:C_Small") (at 238.76 146.05 0) (unit 1)
     (in_bom yes) (on_board yes)
-    (property "Reference" "C?" (id 0) (at 240.03 143.51 0)
+    (property "Reference" "C410" (id 0) (at 240.03 143.51 0)
       (effects (font (size 1.27 1.27)) (justify left))
     )
@@
   (symbol (lib_id "power:GND") (at 241.3 105.41 0) (unit 1)
     (in_bom yes) (on_board yes)
-    (property "Reference" "#PWR?" (id 0) (at 241.3 111.76 0)
+    (property "Reference" "#PWR0405" (id 0) (at 241.3 111.76 0)
       (effects (font (size 1.27 1.27)) hide)
     )
@@
   (symbol (lib_id "Device:C_Small") (at 246.38 146.05 0) (unit 1)
     (in_bom yes) (on_board yes)
-    (property "Reference" "C?" (id 0) (at 247.65 143.51 0)
+    (property "Reference" "C411" (id 0) (at 247.65 143.51 0)
       (effects (font (size 1.27 1.27)) (justify left))
     )
@@
   (symbol (lib_id "Device:C_Polarized_Small_US") (at 228.6 34.29 0) (unit 1)
     (in_bom yes) (on_board yes)
-    (property "Reference" "C?" (id 0) (at 229.87 31.75 0)
+    (property "Reference" "C405" (id 0) (at 229.87 31.75 0)
       (effects (font (size 1.27 1.27)) (justify left))
     )
@@
   (symbol (lib_id "power:GND") (at 234.95 60.96 0) (unit 1)
     (in_bom yes) (on_board yes)
-    (property "Reference" "#PWR?" (id 0) (at 234.95 67.31 0)
+    (property "Reference" "#PWR0404" (id 0) (at 234.95 67.31 0)
       (effects (font (size 1.27 1.27)) hide)
     )
@@
   (symbol (lib_id "Device:C_Small") (at 213.36 146.05 0) (unit 1)
     (in_bom yes) (on_board yes)
-    (property "Reference" "C?" (id 0) (at 214.63 143.51 0)
+    (property "Reference" "C403" (id 0) (at 214.63 143.51 0)
       (effects (font (size 1.27 1.27)) (justify left))
     )
@@
   (symbol (lib_id "Device:C_Small") (at 254 146.05 0) (unit 1)
     (in_bom yes) (on_board yes)
-    (property "Reference" "C?" (id 0) (at 255.27 143.51 0)
+    (property "Reference" "C412" (id 0) (at 255.27 143.51 0)
       (effects (font (size 1.27 1.27)) (justify left))
     )
@@
   (symbol (lib_id "Device:L_Small") (at 229.87 19.05 90) (unit 1)
     (in_bom yes) (on_board yes) (fields_autoplaced)
-    (property "Reference" "L?" (id 0) (at 229.87 13.97 90))
+    (property "Reference" "L401" (id 0) (at 229.87 13.97 90))
     (property "Value" "BLM41PG471SN1L" (id 1) (at 229.87 16.51 90))
     (property "Footprint" "Inductor_SMD:L_1806_4516Metric_Pad1.45x1.90mm_HandSolder" (id 2) (at 229.87 19.05 0)
@@
   (symbol (lib_id "Device:C_Small") (at 198.12 146.05 0) (unit 1)
     (in_bom yes) (on_board yes)
-    (property "Reference" "C?" (id 0) (at 199.39 143.51 0)
+    (property "Reference" "C401" (id 0) (at 199.39 143.51 0)
       (effects (font (size 1.27 1.27)) (justify left))
     )
@@
   (symbol (lib_id "Device:C_Small") (at 234.95 34.29 0) (unit 1)
     (in_bom yes) (on_board yes)
-    (property "Reference" "C?" (id 0) (at 236.22 31.75 0)
+    (property "Reference" "C408" (id 0) (at 236.22 31.75 0)
       (effects (font (size 1.27 1.27)) (justify left))
     )
@@
   (symbol (lib_id "power:GND") (at 234.95 24.13 0) (unit 1)
     (in_bom yes) (on_board yes)
-    (property "Reference" "#PWR?" (id 0) (at 234.95 30.48 0)
+    (property "Reference" "#PWR0402" (id 0) (at 234.95 30.48 0)
       (effects (font (size 1.27 1.27)) hide)
     )
@@
   (symbol (lib_id "Device:C_Small") (at 269.24 146.05 0) (unit 1)
     (in_bom yes) (on_board yes)
-    (property "Reference" "C?" (id 0) (at 270.51 143.51 0)
+    (property "Reference" "C414" (id 0) (at 270.51 143.51 0)
       (effects (font (size 1.27 1.27)) (justify left))
     )
@@
   (symbol (lib_id "Device:C_Small") (at 276.86 146.05 0) (unit 1)
     (in_bom yes) (on_board yes)
-    (property "Reference" "C?" (id 0) (at 278.13 143.51 0)
+    (property "Reference" "C415" (id 0) (at 278.13 143.51 0)
       (effects (font (size 1.27 1.27)) (justify left))
     )
@@
   (symbol (lib_id "Device:C_Small") (at 234.95 21.59 0) (unit 1)
     (in_bom yes) (on_board yes)
-    (property "Reference" "C?" (id 0) (at 236.22 20.32 0)
+    (property "Reference" "C407" (id 0) (at 236.22 20.32 0)
       (effects (font (size 1.27 1.27)) (justify left))
     )
@@
   (symbol (lib_id "power:GND") (at 213.36 152.4 0) (unit 1)
     (in_bom yes) (on_board yes)
-    (property "Reference" "#PWR?" (id 0) (at 213.36 158.75 0)
+    (property "Reference" "#PWR0401" (id 0) (at 213.36 158.75 0)
       (effects (font (size 1.27 1.27)) hide)
     )
@@
   (symbol (lib_id "2022-01-19_19-47-49:ATSAM4E8EA-AN") (at 55.88 30.48 0) (unit 1)
     (in_bom yes) (on_board yes) (fields_autoplaced)
-    (property "Reference" "U?" (id 0) (at 88.9 16.51 0)
+    (property "Reference" "U401" (id 0) (at 88.9 16.51 0)
       (effects (font (size 1.524 1.524)))
     )
@@
   (symbol (lib_id "Device:C_Small") (at 261.62 146.05 0) (unit 1)
     (in_bom yes) (on_board yes)
-    (property "Reference" "C?" (id 0) (at 262.89 143.51 0)
+    (property "Reference" "C413" (id 0) (at 262.89 143.51 0)
       (effects (font (size 1.27 1.27)) (justify left))
     )
@@
   (symbol (lib_id "Device:C_Small") (at 228.6 146.05 0) (unit 1)
     (in_bom yes) (on_board yes)
-    (property "Reference" "C?" (id 0) (at 229.87 143.51 0)
+    (property "Reference" "C406" (id 0) (at 229.87 143.51 0)
       (effects (font (size 1.27 1.27)) (justify left))
     )
@@
   (symbol (lib_id "2022-01-19_19-47-49:ATSAM4E8EA-AN") (at 241.3 27.94 0) (unit 3)
     (in_bom yes) (on_board yes)
-    (property "Reference" "U?" (id 0) (at 259.08 16.51 0)
+    (property "Reference" "U401" (id 0) (at 259.08 16.51 0)
       (effects (font (size 1.524 1.524)) (justify left))
     )
@@
   (symbol (lib_id "Device:C_Small") (at 220.98 146.05 0) (unit 1)
     (in_bom yes) (on_board yes)
-    (property "Reference" "C?" (id 0) (at 222.25 143.51 0)
+    (property "Reference" "C404" (id 0) (at 222.25 143.51 0)
       (effects (font (size 1.27 1.27)) (justify left))
     )
@@
   (symbol (lib_id "power:GND") (at 254 152.4 0) (unit 1)
     (in_bom yes) (on_board yes)
-    (property "Reference" "#PWR?" (id 0) (at 254 158.75 0)
+    (property "Reference" "#PWR0406" (id 0) (at 254 158.75 0)
       (effects (font (size 1.27 1.27)) hide)
     )
@@
   (symbol (lib_id "Device:C_Small") (at 205.74 146.05 0) (unit 1)
     (in_bom yes) (on_board yes)
-    (property "Reference" "C?" (id 0) (at 207.01 143.51 0)
-      (effects (font (size 1.27 1.27)) (justify left))
-    )
+    (property "Reference" "C402" (id 0) (at 207.01 143.51 0)
+      (effects (font (size 1.27 1.27)) (justify left))
+    )
