File: kicad_project/digitizer/ANALOG.kicad_sch (KiCad schematic)
At the start: 18 parts, among them IC301 ADS1234IPWR, J301 T4141012051-000, J302 T4141012051-000, J303 T4141012051-000

Commit message: updated schematic to include terminal blocks for the analog M12 connectors and the downstream CANPWR connector
Parts:
- J301: value T4141012051-000 -> Load Cell 1; footprint CONN5_T4141012051 -> SamacSys_Parts:1935187
- J302: value T4141012051-000 -> Load Cell 3; footprint CONN5_T4141012051 -> SamacSys_Parts:1935187
- J303: value T4141012051-000 -> Load Cell 2; footprint CONN5_T4141012051 -> SamacSys_Parts:1935187
Other:
- moved on the sheet: R307
Changed lines of the file:
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@@
     (stroke (width 0) (type default) (color 0 0 0 0))
   )
-  (wire (pts (xy 156.21 74.93) (xy 158.75 74.93))
+  (wire (pts (xy 156.21 74.93) (xy 161.29 74.93))
     (stroke (width 0) (type default) (color 0 0 0 0))
   )
@@
     (stroke (width 0) (type default) (color 0 0 0 0))
   )
-  (wire (pts (xy 163.83 74.93) (xy 173.99 74.93))
+  (wire (pts (xy 166.37 74.93) (xy 173.99 74.93))
     (stroke (width 0) (type default) (color 0 0 0 0))
   )
@@
       (effects (font (size 1.524 1.524)))
     )
-    (property "Value" "T4141012051-000" (id 1) (at 53.34 46.99 0)
+    (property "Value" "Load Cell 1" (id 1) (at 53.34 46.99 0)
       (effects (font (size 1.524 1.524)))
     )
-    (property "Footprint" "CONN5_T4141012051" (id 2) (at 52.07 55.626 0)
+    (property "Footprint" "SamacSys_Parts:1935187" (id 2) (at 52.07 55.626 0)
       (effects (font (size 1.524 1.524)) hide)
     )
@@
     (pin "1")
   )
-  (symbol (lib_id "Device:R_Small") (at 161.29 74.93 90) (unit 1)
-    (in_bom yes) (on_board yes)
-    (property "Reference" "R307" (id 0) (at 160.02 73.66 90)
-      (effects (font (size 1.27 1.27)) (justify left))
-    )
-    (property "Value" "100" (id 1) (at 167.64 73.66 90)
-      (effects (font (size 1.27 1.27)) (justify left))
-    )
-    (property "Footprint" "Resistor_SMD:R_2512_6332Metric_Pad1.40x3.35mm_HandSolder" (id 2) (at 161.29 74.93 0)
-      (effects (font (size 1.27 1.27)) hide)
-    )
-    (property "Datasheet" "~" (id 3) (at 161.29 74.93 0)
+  (symbol (lib_id "Device:R_Small") (at 163.83 74.93 90) (unit 1)
+    (in_bom yes) (on_board yes)
+    (property "Reference" "R307" (id 0) (at 162.56 73.66 90)
+      (effects (font (size 1.27 1.27)) (justify left))
+    )
+    (property "Value" "100" (id 1) (at 170.18 73.66 90)
+      (effects (font (size 1.27 1.27)) (justify left))
+    )
+    (property "Footprint" "Resistor_SMD:R_2512_6332Metric_Pad1.40x3.35mm_HandSolder" (id 2) (at 163.83 74.93 0)
+      (effects (font (size 1.27 1.27)) hide)
+    )
+    (property "Datasheet" "~" (id 3) (at 163.83 74.93 0)
       (effects (font (size 1.27 1.27)) hide)
     )
@@
       (effects (font (size 1.524 1.524)))
     )
-    (property "Value" "T4141012051-000" (id 1) (at 53.34 85.09 0)
+    (property "Value" "Load Cell 3" (id 1) (at 53.34 85.09 0)
       (effects (font (size 1.524 1.524)))
     )
-    (property "Footprint" "CONN5_T4141012051" (id 2) (at 52.07 93.726 0)
+    (property "Footprint" "SamacSys_Parts:1935187" (id 2) (at 52.07 93.726 0)
       (effects (font (size 1.524 1.524)) hide)
     )
@@
       (effects (font (size 1.524 1.524)))
     )
-    (property "Value" "T4141012051-000" (id 1) (at 53.34 125.73 0)
+    (property "Value" "Load Cell 2" (id 1) (at 53.34 125.73 0)
       (effects (font (size 1.524 1.524)))
     )
-    (property "Footprint" "CONN5_T4141012051" (id 2) (at 52.07 134.366 0)
+    (property "Footprint" "SamacSys_Parts:1935187" (id 2) (at 52.07 134.366 0)
       (effects (font (size 1.524 1.524)) hide)
     )
     (property "Datasheet" "" (id 3) (at 62.23 140.97 0)
-      (effects (font (size 1.524 1.524)))
-    )
-    (pin "1")
+      (effects (font (size 1.524 1.524)) hide)
+    )
+    (pin "1")

Commit message: cleared ALL errors from electrical rules check; had to explicitly define a bunch of pins, and remove a few bugs (shorted lines, etc.)
Parts:
- J302: value Load Cell 3 -> Load Cell 2
- renumbered C305 to C304, C304 to C305
Other:
- moved on the sheet: C305

Commit message: updated a name
Parts:
- J303: value Load Cell 2 -> Load Cell 3
Changed lines of the file:
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@@
       (effects (font (size 1.524 1.524)))
     )
-    (property "Value" "Load Cell 2" (id 1) (at 53.34 125.73 0)
+    (property "Value" "Load Cell 3" (id 1) (at 53.34 125.73 0)
       (effects (font (size 1.524 1.524)))
     )

Commit message: added 5pin term blocks for the M12 connections, so we can properly ground the shield connections
Parts:
- J301, J302, J303: footprint SamacSys_Parts:1935187 -> SamacSys_Parts:1935190
Changed lines of the file:
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@@
       (effects (font (size 1.524 1.524)))
     )
-    (property "Footprint" "SamacSys_Parts:1935187" (id 2) (at 72.39 68.834 0)
+    (property "Footprint" "SamacSys_Parts:1935190" (id 2) (at 72.39 68.834 0)
       (effects (font (size 1.524 1.524)) hide)
     )
@@
       (effects (font (size 1.524 1.524)))
     )
-    (property "Footprint" "SamacSys_Parts:1935187" (id 2) (at 72.39 147.574 0)
+    (property "Footprint" "SamacSys_Parts:1935190" (id 2) (at 72.39 147.574 0)
       (effects (font (size 1.524 1.524)) hide)
     )
@@
       (effects (font (size 1.524 1.524)))
     )
-    (property "Footprint" "SamacSys_Parts:1935187" (id 2) (at 72.39 106.934 0)
+    (property "Footprint" "SamacSys_Parts:1935190" (id 2) (at 72.39 106.934 0)
       (effects (font (size 1.524 1.524)) hide)
     )
