File: kicad_project/digitizer/digitizer.kicad_pcb (KiCad board)
At the start: 2 copper layers, 96 x 74 mm, 63 parts, among them IC201 MAX3059ASA+T UPSTREAM, IC202 MAX6035AAUR50+T, IC203 MAX3059ASA+T DOWNSTREAM, IC204 MAX6043BAUT33+T, IC301 ADS1234IPWR, J201 DT15-4P (UPSTREAM), J202 DT06-4S (DOWNSTREAM), J301 Load Cell 1, J302 Load Cell 2, J303 Load Cell 3, J401 SHF-105-01-L-D-TH-TR, U401 ATSAM4E8EA-AN

Commit message: backup commit; going to change all of the capacitor and resistor sizes to be much smaller
Parts:
- R201: moved to B.Cu
- moved R201 46.9 mm to (105.0, 102.5)
- moved IC201 3.30 mm to (105.3, 97.6)
- moved IC203 3.30 mm to (93.3, 97.6)
Routing:
- net Net-(IC201-Pad8): track 0.00 -> 10.8 mm, vias 0 -> 1
Changed lines of the file:
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@@
   )
   (footprint "Resistor_SMD:R_2512_6332Metric_Pad1.40x3.35mm_HandSolder" (layer "F.Cu")
-    (at 58.07 101.97)
-    (descr "Resistor SMD 2512 (6332 Metric), square (rectangular) end terminal, IPC_7351 nominal with elongated pad for handsoldering. (Body size source: IPC-SM-782 page 72, https://www.pcb-3d.com/wordpress/wp-content/uploads/ipc-sm-782a_amendment_1_and_2.pdf), generated with kicad-footprint-generator")
-    (tags "resistor handsolder")
-    (property "Sheetfile" "CANPWR.kicad_sch")
-    (property "Sheetname" "CANPWR")
-    (attr smd)
-    (fp_text reference "R201" (at 0 -2.62) (layer "F.SilkS")
-      (effects (font (size 1 1) (thickness 0.15)))
-    )
-    (fp_text value "50k" (at 0 2.62) (layer "F.Fab")
-      (effects (font (size 1 1) (thickness 0.15)))
-    )
-    (fp_text user "${REFERENCE}" (at 0 0) (layer "F.Fab")
-      (effects (font (size 1 1) (thickness 0.15)))
-    )
-    (fp_line (start -2.177064 1.71) (end 2.177064 1.71) (layer "F.SilkS") (width 0.12))
-    (fp_line (start -2.177064 -1.71) (end 2.177064 -1.71) (layer "F.SilkS") (width 0.12))
-    (fp_line (start -4 1.92) (end -4 -1.92) (layer "F.CrtYd") (width 0.05))
-    (fp_line (start 4 1.92) (end -4 1.92) (layer "F.CrtYd") (width 0.05))
-    (fp_line (start -4 -1.92) (end 4 -1.92) (layer "F.CrtYd") (width 0.05))
-    (fp_line (start 4 -1.92) (end 4 1.92) (layer "F.CrtYd") (width 0.05))
-    (fp_line (start 3.15 -1.6) (end 3.15 1.6) (layer "F.Fab") (width 0.1))
-    (fp_line (start -3.15 1.6) (end -3.15 -1.6) (layer "F.Fab") (width 0.1))
-    (fp_line (start -3.15 -1.6) (end 3.15 -1.6) (layer "F.Fab") (width 0.1))
-    (fp_line (start 3.15 1.6) (end -3.15 1.6) (layer "F.Fab") (width 0.1))
-    (pad "1" smd roundrect locked (at -3.05 0) (size 1.4 3.35) (layers "F.Cu" "F.Paste" "F.Mask") (roundrect_rratio 0.178571)
-      (net 13 "Net-(IC201-Pad8)") (pintype "passive"))
-    (pad "2" smd roundrect locked (at 3.05 0) (size 1.4 3.35) (layers "F.Cu" "F.Paste" "F.Mask") (roundrect_rratio 0.178571)
-      (net 1 "GND") (pintype "passive"))
-    (model "${KICAD6_3DMODEL_DIR}/Resistor_SMD.3dshapes/R_2512_6332Metric.wrl"
-      (offset (xyz 0 0 0))
-      (scale (xyz 1 1 1))
-      (rotate (xyz 0 0 0))
-    )
-  )
-  (footprint "Resistor_SMD:R_2512_6332Metric_Pad1.40x3.35mm_HandSolder" (layer "F.Cu")
     (at 29.21 84.37)
     (descr "Resistor SMD 2512 (6332 Metric), square (rectangular) end terminal, IPC_7351 nominal with elongated pad for handsoldering. (Body size source: IPC-SM-782 page 72, https://www.pcb-3d.com/wordpress/wp-content/uploads/ipc-sm-782a_amendment_1_and_2.pdf), generated with kicad-footprint-generator")
@@
   )
   (footprint "SamacSys_Parts:SOIC127P600X175-8N" (layer "F.Cu")
-    (at 105.2 94.3)
+    (at 105.3 97.6)
     (descr "S8+4")
     (tags "Integrated Circuit")
@@
   )
   (footprint "SamacSys_Parts:SOIC127P600X175-8N" (layer "F.Cu")
-    (at 93.2 94.3 180)
+    (at 93.3 97.6 180)
     (descr "S8+4")
     (tags "Integrated Circuit")
@@
     )
   )
+  (footprint "Resistor_SMD:R_2512_6332Metric_Pad1.40x3.35mm_HandSolder" (layer "B.Cu")
+    (at 105 102.5)
+    (descr "Resistor SMD 2512 (6332 Metric), square (rectangular) end terminal, IPC_7351 nominal with elongated pad for handsoldering. (Body size source: IPC-SM-782 page 72, https://www.pcb-3d.com/wordpress/wp-content/uploads/ipc-sm-782a_amendment_1_and_2.pdf), generated with kicad-footprint-generator")
+    (tags "resistor handsolder")
+    (property "Sheetfile" "CANPWR.kicad_sch")
+    (property "Sheetname" "CANPWR")
+    (attr smd)
+    (fp_text reference "R201" (at 0 2.62) (layer "B.SilkS")
+      (effects (font (size 1 1) (thickness 0.15)) (justify mirror))
+    )
+    (fp_text value "50k" (at 0 -2.62) (layer "B.Fab")
+      (effects (font (size 1 1) (thickness 0.15)) (justify mirror))
+    )
+    (fp_text user "${REFERENCE}" (at 0 0) (layer "B.Fab")
+      (effects (font (size 1 1) (thickness 0.15)) (justify mirror))
+    )
+    (fp_line (start -2.177064 -1.71) (end 2.177064 -1.71) (layer "B.SilkS") (width 0.12))
+    (fp_line (start -2.177064 1.71) (end 2.177064 1.71) (layer "B.SilkS") (width 0.12))
+    (fp_line (start -4 -1.92) (end -4 1.92) (layer "B.CrtYd") (width 0.05))
+    (fp_line (start 4 -1.92) (end -4 -1.92) (layer "B.CrtYd") (width 0.05))
+    (fp_line (start -4 1.92) (end 4 1.92) (layer "B.CrtYd") (width 0.05))
+    (fp_line (start 4 1.92) (end 4 -1.92) (layer "B.CrtYd") (width 0.05))
+    (fp_line (start 3.15 1.6) (end 3.15 -1.6) (layer "B.Fab") (width 0.1))
+    (fp_line (start -3.15 -1.6) (end -3.15 1.6) (layer "B.Fab") (width 0.1))
+    (fp_line (start -3.15 1.6) (end 3.15 1.6) (layer "B.Fab") (width 0.1))
+    (fp_line (start 3.15 -1.6) (end -3.15 -1.6) (layer "B.Fab") (width 0.1))
+    (pad "1" smd roundrect locked (at -3.05 0) (size 1.4 3.35) (layers "B.Cu" "B.Paste" "B.Mask") (roundrect_rratio 0.178571)
+      (net 13 "Net-(IC201-Pad8)") (pintype "passive"))
+    (pad "2" smd roundrect locked (at 3.05 0) (size 1.4 3.35) (layers "B.Cu" "B.Paste" "B.Mask") (roundrect_rratio 0.178571)
+      (net 1 "GND") (pintype "passive"))
+    (model "${KICAD6_3DMODEL_DIR}/Resistor_SMD.3dshapes/R_2512_6332Metric.wrl"
+      (offset (xyz 0 0 0))
+      (scale (xyz 1 1 1))
+      (rotate (xyz 0 0 0))
+    )
+  )
   (footprint "Capacitor_SMD:C_2220_5650Metric_Pad1.97x5.40mm_HandSolder" (layer "B.Cu")
     (at 116 105 -90)
@@
   (via (at 116 105.3005) (size 0.8) (drill 0.4) (layers "F.Cu" "B.Cu") (net 5))
   (segment (start 116 107.6375) (end 116 105.3005) (width 0.25) (layer "B.Cu") (net 5))
+  (segment (start 105 101.5) (end 104 102.5) (width 0.25) (layer "F.Cu") (net 13))
+  (segment (start 107.5745 95.695) (end 105 98.2695) (width 0.25) (layer "F.Cu") (net 13))
+  (segment (start 105 98.2695) (end 105 101.5) (width 0.25) (layer "F.Cu") (net 13))
+  (segment (start 104 102.5) (end 101.95 102.5) (width 0.25) (layer "F.Cu") (net 13))
+  (segment (start 108.012 95.695) (end 107.5745 95.695) (width 0.25) (layer "F.Cu") (net 13))
+  (via (at 101.95 102.5) (size 0.8) (drill 0.4) (layers "F.Cu" "B.Cu") (net 13))
   (segment (start 120.312 103.425) (end 119.350478 103.425) (width 0.25) (layer "F.Cu") (net 22))
   (segment (start 115.7 99.774522) (end 115.7 92.95) (width 0.25) (layer "F.Cu") (net 22))

Commit message: updated schematic to use all 0805 parts (both caps and resistors)
Parts:
- R403, R404: footprint Resistor_SMD:R_2512_6332Metric_Pad1.40x3.35mm_HandSolder -> Resistor_SMD:R_0805_2012Metric_Pad1.20x1.40mm_HandSolder

Commit message: updated layout with new, smaller passive components
Parts:
- C201, C202, C203, C301, C302, C303, C304, C305, C306, C307, C401, C403, C404, C405, C406, C407, C408, C409, C410, C411, C412, C413, C414, C415, C416: footprint Capacitor_SMD:C_2220_5650Metric_Pad1.97x5.40mm_HandSolder -> Capacitor_SMD:C_0805_2012Metric_Pad1.18x1.45mm_HandSolder
- C204: footprint Capacitor_SMD:C_2220_5650Metric_Pad1.97x5.40mm_HandSolder -> Capacitor_SMD:C_0805_2012Metric_Pad1.18x1.45mm_HandSolder; moved to F.Cu
- C402: footprint Capacitor_Tantalum_SMD:CP_EIA-6032-20_AVX-F_Pad2.25x2.35mm_HandSolder -> Capacitor_SMD:C_0805_2012Metric_Pad1.18x1.45mm_HandSolder
- R201, R203, R301, R302, R303, R304, R305, R306, R307, R401, R402, R405, R406, R407: footprint Resistor_SMD:R_2512_6332Metric_Pad1.40x3.35mm_HandSolder -> Resistor_SMD:R_0805_2012Metric_Pad1.20x1.40mm_HandSolder
- R202: footprint Resistor_SMD:R_2512_6332Metric_Pad1.40x3.35mm_HandSolder -> Resistor_SMD:R_0805_2012Metric_Pad1.20x1.40mm_HandSolder; moved to B.Cu
- moved R202 47.8 mm to (98.8, 95.8), turned to 180 degrees
- moved R301 9.68 mm to (115.5, 99.2)
- moved R302 9.24 mm to (118.0, 99.2)
- moved R201 9.03 mm to (111.0, 95.8)
- moved R203 4.12 mm to (95.5, 56.0)
- moved R303 3.41 mm to (135.8, 97.8)
- moved C204 3.25 mm to (112.8, 56.0)
- moved R305 2.97 mm to (132.5, 97.8)
- moved R304 2.80 mm to (129.2, 97.8)
- moved IC202 2.65 mm to (163.2, 96.2), turned to 0 degrees
- moved C304 2.50 mm to (147.4, 116.5)
- moved C301 2.20 mm to (123.2, 97.5)
- moved C306 2.01 mm to (80.0, 105.3)
- moved C307 2.00 mm to (113.5, 117.0)
- moved IC204 1.00 mm to (117.0, 56.0)
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Routing:
- net /CANPWR/CANH_DOWNSTREAM: track 0.00 -> 39.3 mm, vias 0 -> 1
- net /CANPWR/CANL_DOWNSTREAM: track 0.00 -> 35.7 mm, vias 0 -> 1
- net ADC_MUX_0: track 25.0 -> 37.4 mm
- net ADC_MUX_1: track 27.6 -> 38.9 mm
- net Net-(IC301-Pad8): track 15.2 -> 6.40 mm
- net Net-(IC201-Pad8): track 10.8 -> 2.01 mm
- net Net-(IC301-Pad7): track 12.9 -> 4.71 mm
- net 12V_CLEAN: track 64.9 -> 69.4 mm, vias 2 -> 1
- net GND: track 32.5 -> 28.5 mm, vias 4 -> 3
- net Net-(IC301-Pad26): track 12.7 -> 10.4 mm
- net I2C_SDA: track 29.8 -> 32.0 mm
- net /ANALOG/load cell 3 - signal (+): track 26.9 -> 24.9 mm
- net /ANALOG/load cell 3 - signal (-): track 31.6 -> 29.7 mm
- net Net-(IC203-Pad8): track 0.00 -> 1.76 mm, vias 0 -> 1
- net /ANALOG/load cell 1 - signal (-): track 42.9 -> 41.3 mm
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